File: Hardware/PCB/Andy_PCB_5.0.0/MothBox/GPS.kicad_sch (KiCad schematic)
At the start: 26 parts, among them U1 Days, U17 GPs 5 pin PM2.54-1*5, U2 Hours1, U20 74HC165, U21 74HC165, U22 74HC165, U6 Hours2, U7 Modes, U8 74HC165, U9 74HC165

Commit message: Tidied up and merged with local main
Other:
- note added: "This could be changed to use both nibbles. v5.1 would be Bunary 01010001, Hex 0x51"
Changed lines of the file:
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@@
+		)
+	)
+	(text "This could be changed to use both nibbles.\nv5.1 would be Bunary 01010001, Hex 0x51"
+		(exclude_from_sim no)
+		(at 105.41 208.026 0)
+		(effects
+			(font
+				(size 1.27 1.27)
+				(thickness 0.254)
+				(bold yes)
+			)
 		)
 	)
