File: Hardware/PCB/Andy_PCB_5.0.0/MothBox/MothBox.kicad_pcb (KiCad board)
At the start: 2 copper layers, 237 x 140.5 mm, 163 parts, among them P1 Raw Input, P2 12V Regulated Input, P3 Input to regulator, P4 External Attractor, Q1 BC817, Q10 BC817, Q11 BC817, Q2 SUD50P06-15-GE3, Q4 BC817, Q5 SUD50P06-15-GE3, Q6 BC817, Q7 SUD50P06-15-GE3, Q8 BC817, Q9 BC817, U1 Days, U10 FDS4435BZ, U11 FDS4435BZ, U12 FDS4435BZ, U13 FDS4435BZ, U16 Female Inv Socket Pi 2.54-2*20, U17 GPs 5 pin PM2.54-1*5, U18 RASPBERRY_PI_4B_4GB, U19 INA219BIDCNT, U2 Hours1, U20 74HC165, U21 74HC165, U22 74HC165, U3 XL4015E1, U5 RASPBERRY_PI_5, U6 Hours2, U7 Modes, U8 74HC165, U9 74HC165

Commit message: Tidied up and merged with local main
Parts:
- moved R66 1.43 mm to (234.1, 123.1), turned to 180 degrees
Routing:
- net /Photo LED's/+12V_L_LED: track 335.9 -> 330.6 mm
- net +12V: track 466.8 -> 462.4 mm
- net GPS_PPS: track 115.9 -> 119.2 mm
- net GPS_TX: track 157.9 -> 157.1 mm
